File: PCB/hackpad.kicad_pcb (KiCad board)
At the start: 2 copper layers, 92.9 x 83.8 mm, 30 parts, among them J1 Conn_01x04_Pin, SW1 SW_Push_45deg, SW10 SW_Push_45deg, SW11 SW_Push_45deg, SW12 SW_Push_45deg, SW14 SW_Push, SW15 SW_Push, SW2 SW_Push_45deg, SW3 SW_Push_45deg, SW4 SW_Push_45deg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

Commit message: fixed pcb picture + label
Other:
- board text added: "BEETLEPAD"
- board text removed: "ISABELLE"
Changed lines of the file:
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@@
 		)
 	)
-	(gr_text "ISABELLE\n"
+	(gr_text "BEETLEPAD\n"
 		(at 90.298463 102.5525 0)
 		(layer "B.SilkS")
